Commit message: complete urdf

File: urdfgripper_description/urdf/materials.xacro (robot description, xacro)
@@ -1,6 +1,6 @@
 <?xml version="1.0" ?>
 <robot name="urdfgripper" xmlns:xacro="http://www.ros.org/wiki/xacro" >
-<material name="silver">
-  <color rgba="0.700 0.700 0.700 1.000"/>
+<material name="cyan">
+  <color rgba="0.000 1.000 0.950 1.000"/>
 </material>
 </robot>

File: urdfgripper_description/urdf/urdfgripper.xacro (robot description, xacro)
@@ -4,5 +4,5 @@
 <xacro:include filename="$(find urdfgripper_description)/urdf/urdfgripper.trans" />
 <xacro:include filename="$(find urdfgripper_description)/urdf/urdfgripper.gazebo" />
-<link name="base_link">
+<link name="gripper_base_link">
   <inertial>
     <origin xyz="1.9099884677715165e-13 -8.588463814791657e-18 0.050480059207214864" rpy="0 0 0"/>
@@ -15,5 +15,5 @@
       <mesh filename="package://urdfgripper_description/meshes/base_link.stl" scale="0.001 0.001 0.001"/>
     </geometry>
-    <material name="silver"/>
+    <material name="cyan"/>
   </visual>
   <collision>
@@ -35,5 +35,5 @@
       <mesh filename="package://urdfgripper_description/meshes/clamp2_1.stl" scale="0.001 0.001 0.001"/>
     </geometry>
-    <material name="silver"/>
+    <material name="cyan"/>
   </visual>
   <collision>
@@ -55,5 +55,5 @@
       <mesh filename="package://urdfgripper_description/meshes/joint_gripper2_1.stl" scale="0.001 0.001 0.001"/>
     </geometry>
-    <material name="silver"/>
+    <material name="cyan"/>
   </visual>
   <collision>
@@ -75,5 +75,5 @@
       <mesh filename="package://urdfgripper_description/meshes/clamp1_1.stl" scale="0.001 0.001 0.001"/>
     </geometry>
-    <material name="silver"/>
+    <material name="cyan"/>
   </visual>
   <collision>
@@ -95,5 +95,5 @@
       <mesh filename="package://urdfgripper_description/meshes/joint_gripper1_1.stl" scale="0.001 0.001 0.001"/>
     </geometry>
-    <material name="silver"/>
+    <material name="cyan"/>
   </visual>
   <collision>
@@ -115,5 +115,5 @@
       <mesh filename="package://urdfgripper_description/meshes/joint_gripper3_1.stl" scale="0.001 0.001 0.001"/>
     </geometry>
-    <material name="silver"/>
+    <material name="cyan"/>
   </visual>
   <collision>
@@ -135,5 +135,5 @@
       <mesh filename="package://urdfgripper_description/meshes/joint_gripper1_1.stl" scale="0.001 0.001 0.001"/>
     </geometry>
-    <material name="silver"/>
+    <material name="cyan"/>
   </visual>
   <collision>
@@ -155,5 +155,5 @@
       <mesh filename="package://urdfgripper_description/meshes/joint_gripper2_1.stl" scale="0.001 0.001 0.001"/>
     </geometry>
-    <material name="silver"/>
+    <material name="cyan"/>
   </visual>
   <collision>
@@ -164,35 +164,35 @@
   </collision>
 </link>
-<joint name="Revolute 1" type="continuous">
+<joint name="Revolute_1" type="continuous">
   <origin xyz="-0.036 -0.01325 0.1238" rpy="0 -0.84 0"/>
-  <parent link="base_link"/>
+  <parent link="gripper_base_link"/>
   <child link="clamp2_1"/>
   <axis xyz="0.0 -1.0 0.0"/>
-  <mimic joint="Slider 5" multiplier="62.0" offset="0.0"/>
-</joint>
-<joint name="Revolute 2" type="continuous">
+  <mimic joint="Slider_5" multiplier="62.0" offset="0.0"/>
+</joint>
+<joint name="Revolute_2" type="continuous">
   <origin xyz="-0.018 -0.007 -0.023" rpy="0 -0.07 0"/>
   <parent link="joint_gripper3_1"/>
   <child link="joint_gripper2_2"/>
   <axis xyz="0.0 -1.0 -0.0"/>
-  <mimic joint="Slider 5" multiplier="10.0" offset="0.0"/>
-</joint>
-<joint name="Revolute 3" type="continuous">
+  <mimic joint="Slider_5" multiplier="10.0" offset="0.0"/>
+</joint>
+<joint name="Revolute_3" type="continuous">
   <origin xyz="0.036 -0.01325 0.1238" rpy="0 1.74 0"/>
-  <parent link="base_link"/>
+  <parent link="gripper_base_link"/>
   <child link="clamp1_1"/>
   <axis xyz="0.0 -1.0 0.0"/>
-  <mimic joint="Slider 5" multiplier="-62.0" offset="0.0"/>
-</joint>
-<joint name="Revolute 4" type="continuous">
+  <mimic joint="Slider_5" multiplier="-62.0" offset="0.0"/>
+</joint>
+<joint name="Revolute_4" type="continuous">
   <origin xyz="0.018 0.000 -0.023" rpy="0 0.58 0"/>
   <parent link="joint_gripper3_1"/>
   <child link="joint_gripper2_1"/>
   <axis xyz="0.0 -1.0 0.0"/>
-  <mimic joint="Slider 5" multiplier="-10.0" offset="0.0"/>
-</joint>
-<joint name="Slider 5" type="prismatic">
+  <mimic joint="Slider_5" multiplier="-10.0" offset="0.0"/>
+</joint>
+<joint name="Slider_5" type="prismatic">
   <origin xyz="0.0 0.0 0.1410" rpy="0 0 0"/>
-  <parent link="base_link"/>
+  <parent link="gripper_base_link"/>
   <child link="joint_gripper3_1"/>
   <axis xyz="0.0 0.0 1.0"/>

File: walkie3_description/urdf/materials.xacro (robot description, xacro)
@@ -1,6 +1,6 @@
 <?xml version="1.0" ?>
 <robot name="walkie3" xmlns:xacro="http://www.ros.org/wiki/xacro" >
-<material name="silver">
-  <color rgba="0.700 0.700 0.700 1.000"/>
+<material name="black">
+  <color rgba="0.3 0.3 0.3 1.000"/>
 </material>
 </robot>

File: walkie3_description/urdf/walkie3.xacro (robot description, xacro)
@@ -13,12 +13,12 @@
     <origin xyz="0 0 0" rpy="0 0 0"/>
     <geometry>
-      <mesh filename="package://walkie3_description/meshes/base_link.stl" scale="0.001 0.001 0.001"/>
-    </geometry>
-    <material name="silver"/>
+      <mesh filename="package://walkie3_description/meshes/base_link_5cm.stl" scale="0.001 0.001 0.001"/>
+    </geometry>
+    <material name="black"/>
   </visual>
   <collision>
     <origin xyz="0 0 0" rpy="0 0 0"/>
     <geometry>
-      <mesh filename="package://walkie3_description/meshes/base_link.stl" scale="0.001 0.001 0.001"/>
+      <mesh filename="package://walkie3_description/meshes/base_link_5cm.stl" scale="0.001 0.001 0.001"/>
     </geometry>
   </collision>
@@ -35,5 +35,5 @@
       <mesh filename="package://walkie3_description/meshes/rm_1.stl" scale="0.001 0.001 0.001"/>
     </geometry>
-    <material name="silver"/>
+    <material name="black"/>
   </visual>
   <collision>
@@ -55,5 +55,5 @@
       <mesh filename="package://walkie3_description/meshes/lm_1.stl" scale="0.001 0.001 0.001"/>
     </geometry>
-    <material name="silver"/>
+    <material name="black"/>
   </visual>
   <collision>
@@ -75,5 +75,5 @@
       <mesh filename="package://walkie3_description/meshes/front_lidar_1.stl" scale="0.001 0.001 0.001"/>
     </geometry>
-    <material name="silver"/>
+    <material name="black"/>
   </visual>
   <collision>
@@ -95,5 +95,5 @@
       <mesh filename="package://walkie3_description/meshes/back_lidar_1.stl" scale="0.001 0.001 0.001"/>
     </geometry>
-    <material name="silver"/>
+    <material name="black"/>
   </visual>
   <collision>
@@ -115,5 +115,5 @@
       <mesh filename="package://walkie3_description/meshes/lift_1.stl" scale="0.001 0.001 0.001"/>
     </geometry>
-    <material name="silver"/>
+    <material name="black"/>
   </visual>
   <collision>
@@ -135,5 +135,5 @@
       <mesh filename="package://walkie3_description/meshes/camera_case_1.stl" scale="0.001 0.001 0.001"/>
     </geometry>
-    <material name="silver"/>
+    <material name="black"/>
   </visual>
   <collision>
@@ -155,5 +155,5 @@
       <mesh filename="package://walkie3_description/meshes/zed2i_1.stl" scale="0.001 0.001 0.001"/>
     </geometry>
-    <material name="silver"/>
+    <material name="black"/>
   </visual>
   <collision>

File: walkie3_description/urdf/walkie_cr3.xacro (robot description, xacro)
@@ -3,4 +3,5 @@
 <xacro:include filename="$(find walkie3_description)/urdf/walkie3.xacro"/>
 <xacro:include filename="$(find dobot_description)/urdf/cr3_robot.urdf"/>
+<xacro:include filename="$(find urdfgripper_description)/urdf/urdfgripper.xacro"/>
 <link name="virtual_lidar"/>
 <joint name="virtual_lidar_joint" type="fixed">
@@ -14,9 +15,20 @@
     <child  link="dummy_link" />
 </joint>
-<!-- <joint name="zed2i_joint" type="fixed">
+<joint name="cr3_to_gripper" type="fixed">
+    <origin xyz="0.00 0.00 0.00" rpy="0 0 0.785"/>
+    <parent link="Link6" />
+    <child  link="gripper_base_link" />
+</joint>
+<link name="eff"/>
+<joint name="eff_joint" type="fixed">
+  <origin xyz="0.0 0.0 0.18" rpy="0 -1.57 1.57"/>
+  <parent link="gripper_base_link"/>
+  <child link="eff"/>
+</joint>
+ <joint name="zed2i_joint" type="fixed">
     <origin xyz="0.031804 0.09 -0.015" rpy="0 0 0"/>
     <parent link="camera_servo" />
     <child  link="zed2i_base_link" />
-</joint> -->
+</joint>
 <xacro:arg name="camera_name"   default="zed2i" />
 <xacro:arg name="camera_model"  default="zed2i" />
